Commit message: Hokuyo is placed onto minik

File: ros/hokuyo_ws/src/hokuyo_plus/config/gazebo_tama_minik.urdf (robot description, URDF)
Before this commit: robot tama, 6 links, 5 joints
Links:
- removed link world
- added link link_chassis, mass 2; collision box size=0.3 0.3 0.3; collision sphere radius=0.03
- added link link_left_wheel, mass 0.2; collision cylinder length=0.04 radius=0.06; visual cylinder length=0.04 radius=0.06
- added link link_right_wheel, mass 0.2; collision cylinder length=0.04 radius=0.06; visual cylinder length=0.04 radius=0.06
Joints:
- removed joint virtual_joint
- added joint joint_left_wheel: type continuous, parent link_chassis, child link_left_wheel, origin xyz=0 0.2 -0.19 rpy=0 0 0, axis 0 1 0, limit effort=10000 velocity=1000
- added joint joint_right_wheel: type continuous, parent link_chassis, child link_right_wheel, origin xyz=0 -0.2 -0.19 rpy=0 0 0, axis 0 1 0, limit effort=10000 velocity=1000
- added joint joint_sensor_laser: type fixed, parent link_chassis, child taban, origin xyz=0.1 0 0.1 rpy=0 0 0
